Commit message: Implement atomic walking tasks (Leg Lift, Multi-Leg, Static Gait) and training infrastructure

File: Hexapod-ROS/crab_description/hexapod_pybullet.urdf (robot description, URDF)
Before this commit: robot crab, 32 links, 31 joints
Links:
- link coxa_l1: mass 0.1 -> 0.25
- link coxa_l2: mass 0.1 -> 0.25
- link coxa_l3: mass 0.1 -> 0.25
- link coxa_r1: mass 0.1 -> 0.25
- link coxa_r2: mass 0.1 -> 0.25
- link coxa_r3: mass 0.1 -> 0.25
- link femur_l1: mass 0.1 -> 0.25
- link femur_l2: mass 0.1 -> 0.25
- link femur_l3: mass 0.1 -> 0.25
- link femur_r1: mass 0.1 -> 0.25
- link femur_r2: mass 0.1 -> 0.25
- link femur_r3: mass 0.1 -> 0.25
- link tibia_l1: mass 0.1 -> 0.25
- link tibia_l2: mass 0.1 -> 0.25
- link tibia_l3: mass 0.1 -> 0.25
- link tibia_r1: mass 0.1 -> 0.25
- link tibia_r2: mass 0.1 -> 0.25
- link tibia_r3: mass 0.1 -> 0.25
